File: Electronics/digit_board/digit_board.kicad_pcb (KiCad board)
At the start: 2 copper layers, 57.8 x 22.9 mm, 2 parts, among them P1 LED_DISPLAY

Commit message: Updates
Routing:
- net /DEC: track 41.8 -> 38.6 mm
- net /F: track 37.4 -> 34.9 mm
- net /E: track 38.3 -> 36.0 mm
- net /COL: track 42.2 -> 40.0 mm
- net /COL_AN: track 65.6 -> 63.8 mm
- net /G: track 23.0 -> 21.9 mm
- net /DEC_AN: track 62.2 -> 61.2 mm
- net /B: track 23.3 -> 22.5 mm
- net /D: track 37.5 -> 36.9 mm
- net /DIG1: track 19.9 -> 19.4 mm
